Commit message: Add files via upload

File: robot_base_description/urdf/materials.xacro (robot description, xacro)
@@ -16,3 +16,12 @@
   <color rgba="0.7490196078431373 0.7490196078431373 0.7490196078431373 1.0"/>
 </material>
+<material name="iron">
+  <color rgba="0.700 0.700 0.700 1.000"/>
+</material>
+<material name="blue">
+  <color rgba="0.200 0.000 0.700 1.000"/>
+</material>
+<material name="black">
+  <color rgba="0 0 0 1"/>
+</material>
 </robot>

File: robot_base_description/urdf/robot_base.xacro (robot description, xacro)
@@ -1,13 +1,9 @@
 <?xml version="1.0" ?>
-<robot name="robot_base" xmlns:xacro="http://www.ros.org/wiki/xacro">
+<robot name="hoverboard_robot" xmlns:xacro="http://www.ros.org/wiki/xacro">
 <xacro:include filename="$(find robot_base_description)/urdf/materials.xacro" />
-<!-- <xacro:include filename="$(find robot_base_description)/urdf/robot_base.trans" /> -->
+<xacro:include filename="$(find robot_base_description)/urdf/macros.xacro" />
+<xacro:include filename="$(find robot_base_description)/urdf/ros2_control.xacro" />
 <xacro:include filename="$(find robot_base_description)/urdf/robot_base.gazebo" />
 <link name="base_link">
-  <inertial>
-    <origin xyz="0.006873944780110744 4.580236914566031e-07 0.1220357378331037" rpy="0 0 0"/>
-    <mass value="40.16017107067584"/>
-    <inertia ixx="0.955104" iyy="1.642374" izz="2.413188" ixy="-0.000378" iyz="-0.000123" ixz="0.010792"/>
-  </inertial>
   <visual>
     <origin xyz="0 0 0" rpy="0 0 0"/>
@@ -15,5 +11,5 @@
       <mesh filename="file://$(find robot_base_description)/meshes/base_link.stl" scale="0.001 0.001 0.001"/>
     </geometry>
-    <material name="steel_satin"/>
+    <material name="blue"/>
   </visual>
   <collision>
@@ -35,5 +31,5 @@
       <mesh filename="file://$(find robot_base_description)/meshes/left_front_wheel.stl" scale="0.001 0.001 0.001"/>
     </geometry>
-    <material name="opaque252525"/>
+    <material name="black"/>
   </visual>
   <collision>
@@ -55,5 +51,5 @@
       <mesh filename="file://$(find robot_base_description)/meshes/left_back_wheel.stl" scale="0.001 0.001 0.001"/>
     </geometry>
-    <material name="opaque252525"/>
+    <material name="black"/>
   </visual>
   <collision>
@@ -75,5 +71,5 @@
       <mesh filename="file://$(find robot_base_description)/meshes/right_front_wheel.stl" scale="0.001 0.001 0.001"/>
     </geometry>
-    <material name="opaque252525"/>
+    <material name="black"/>
   </visual>
   <collision>
@@ -95,5 +91,5 @@
       <mesh filename="file://$(find robot_base_description)/meshes/right_back_wheel.stl" scale="0.001 0.001 0.001"/>
     </geometry>
-    <material name="opaque252525"/>
+    <material name="black"/>
   </visual>
   <collision>
@@ -115,5 +111,5 @@
       <mesh filename="file://$(find robot_base_description)/meshes/lidar.stl" scale="0.001 0.001 0.001"/>
     </geometry>
-    <material name="steel_satin"/>
+    <material name="black"/>
   </visual>
   <collision>
@@ -135,5 +131,5 @@
       <mesh filename="file://$(find robot_base_description)/meshes/jetson.stl" scale="0.001 0.001 0.001"/>
     </geometry>
-    <material name="opaque252525"/>
+    <material name="black"/>
   </visual>
   <collision>
@@ -155,5 +151,5 @@
       <mesh filename="file://$(find robot_base_description)/meshes/imu.stl" scale="0.001 0.001 0.001"/>
     </geometry>
-    <material name="opaque252525"/>
+    <material name="black"/>
   </visual>
   <collision>
@@ -175,5 +171,5 @@
       <mesh filename="file://$(find robot_base_description)/meshes/front_plate.stl" scale="0.001 0.001 0.001"/>
     </geometry>
-    <material name="steel_satin"/>
+    <material name="blue"/>
   </visual>
   <collision>
@@ -195,5 +191,5 @@
       <mesh filename="file://$(find robot_base_description)/meshes/rear_plate.stl" scale="0.001 0.001 0.001"/>
     </geometry>
-    <material name="steel_satin"/>
+    <material name="blue"/>
   </visual>
   <collision>
@@ -215,5 +211,5 @@
       <mesh filename="file://$(find robot_base_description)/meshes/right_plate.stl" scale="0.001 0.001 0.001"/>
     </geometry>
-    <material name="steel_satin"/>
+    <material name="blue"/>
   </visual>
   <collision>
@@ -235,5 +231,5 @@
       <mesh filename="file://$(find robot_base_description)/meshes/left_plate.stl" scale="0.001 0.001 0.001"/>
     </geometry>
-    <material name="steel_satin"/>
+    <material name="blue"/>
   </visual>
   <collision>
@@ -255,5 +251,5 @@
       <mesh filename="file://$(find robot_base_description)/meshes/top_cover.stl" scale="0.001 0.001 0.001"/>
     </geometry>
-    <material name="steel_satin"/>
+    <material name="blue"/>
   </visual>
   <collision>
@@ -267,18 +263,898 @@
   <inertial>
     <origin xyz="-2.883374428108709e-09 -2.8580817870224923e-09 5.000000000421334e-07" rpy="0 0 0"/>
-    <mass value="0.00013256683868399403"/>
-    <inertia ixx="0.0" iyy="0.0" izz="0.0" ixy="0.0" iyz="-0.0" ixz="0.0"/>
-  </inertial>
-  <visual>
-    <origin xyz="0.0 0.0 -0.2225" rpy="0 0 0"/>
-    <geometry>
-      <mesh filename="file://$(find robot_base_description)/meshes/mount_link.stl" scale="0.001 0.001 0.001"/>
-    </geometry>
-    <material name="steel_satin"/>
-  </visual>
-  <collision>
-    <origin xyz="0.0 0.0 -0.2225" rpy="0 0 0"/>
-    <geometry>
-      <mesh filename="file://$(find robot_base_description)/meshes/mount_link.stl" scale="0.001 0.001 0.001"/>
+    <mass value="2.5346787978702183"/>
+    <inertia ixx="0.005207" iyy="0.005207" izz="0.009019" ixy="-0.0" iyz="-0.0" ixz="0.0"/>
+  </inertial>
+  <visual>
+    <origin xyz="0 0 0" rpy="0 0 0"/>
+    <geometry>
+      <mesh filename="file://$(find arm_description)/meshes/mount_link.stl" scale="0.001 0.001 0.001"/>
+    </geometry>
+    <material name="blue"/>
+  </visual>
+  <collision>
+    <origin xyz="0 0 0" rpy="0 0 0"/>
+    <geometry>
+      <mesh filename="file://$(find arm_description)/meshes/mount_link.stl" scale="0.001 0.001 0.001"/>
+    </geometry>
+  </collision>
+</link>
+<link name="pulley_c_v9_1">
+  <inertial>
+    <origin xyz="-5.567313502074602e-17 4.098862764811248e-17 -0.003294330259347028" rpy="0 0 0"/>
+    <mass value="0.05283781710784995"/>
+    <inertia ixx="2.4e-05" iyy="2.4e-05" izz="3.8e-05" ixy="-0.0" iyz="0.0" ixz="-0.0"/>
+  </inertial>
+  <visual>
+    <origin xyz="-0.0 -0.0 -0.09" rpy="0 0 0"/>
+    <geometry>
+      <mesh filename="file://$(find arm_description)/meshes/pulley_c_v9_1.stl" scale="0.001 0.001 0.001"/>
+    </geometry>
+    <material name="iron"/>
+  </visual>
+  <collision>
+    <origin xyz="-0.0 -0.0 -0.09" rpy="0 0 0"/>
+    <geometry>
+      <mesh filename="file://$(find arm_description)/meshes/pulley_c_v9_1.stl" scale="0.001 0.001 0.001"/>
+    </geometry>
+  </collision>
+</link>
+<link name="shoulder_bearling_house_prt1_v14_1">
+  <inertial>
+    <origin xyz="4.208209917286061e-06 2.4287672297167474e-06 -0.012900153986197746" rpy="0 0 0"/>
+    <mass value="0.057783249767342296"/>
+    <inertia ixx="3.6e-05" iyy="3.6e-05" izz="7.1e-05" ixy="-0.0" iyz="0.0" ixz="0.0"/>
+  </inertial>
+  <visual>
+    <origin xyz="-0.0 -0.0 -0.123" rpy="0 0 0"/>
+    <geometry>
+      <mesh filename="file://$(find arm_description)/meshes/shoulder_bearling_house_prt1_v14_1.stl" scale="0.001 0.001 0.001"/>
+    </geometry>
+    <material name="blue"/>
+  </visual>
+  <collision>
+    <origin xyz="-0.0 -0.0 -0.123" rpy="0 0 0"/>
+    <geometry>
+      <mesh filename="file://$(find arm_description)/meshes/shoulder_bearling_house_prt1_v14_1.stl" scale="0.001 0.001 0.001"/>
+    </geometry>
+  </collision>
+</link>
+<link name="table1_v2_1">
+  <inertial>
+    <origin xyz="-0.01893394777000812 -0.0198227756761575 0.008078541713728321" rpy="0 0 0"/>
+    <mass value="0.9953039551471342"/>
+    <inertia ixx="0.002494" iyy="0.002414" izz="0.004866" ixy="-9.6e-05" iyz="2e-06" ixz="-1e-06"/>
+  </inertial>
+  <visual>
+    <origin xyz="-0.0 -0.0 -0.1344" rpy="0 0 0"/>
+    <geometry>
+      <mesh filename="file://$(find arm_description)/meshes/table1_v2_1.stl" scale="0.001 0.001 0.001"/>
+    </geometry>
+    <material name="blue"/>
+  </visual>
+  <collision>
+    <origin xyz="-0.0 -0.0 -0.1344" rpy="0 0 0"/>
+    <geometry>
+      <mesh filename="file://$(find arm_description)/meshes/table1_v2_1.stl" scale="0.001 0.001 0.001"/>
+    </geometry>
+  </collision>
+</link>
+<link name="shoulder_bearling_house_prt3_v2_1">
+  <inertial>
+    <origin xyz="-3.326885494954389e-06 -9.453818210990768e-11 0.004385481296303423" rpy="0 0 0"/>
+    <mass value="0.05938208856291772"/>
+    <inertia ixx="3.7e-05" iyy="3.7e-05" izz="7.3e-05" ixy="0.0" iyz="-0.0" ixz="-0.0"/>
+  </inertial>
+  <visual>
+    <origin xyz="-0.0 -0.0 -0.1504" rpy="0 0 0"/>
+    <geometry>
+      <mesh filename="file://$(find arm_description)/meshes/shoulder_bearling_house_prt3_v2_1.stl" scale="0.001 0.001 0.001"/>
+    </geometry>
+    <material name="blue"/>
+  </visual>
+  <collision>
+    <origin xyz="-0.0 -0.0 -0.1504" rpy="0 0 0"/>
+    <geometry>
+      <mesh filename="file://$(find arm_description)/meshes/shoulder_bearling_house_prt3_v2_1.stl" scale="0.001 0.001 0.001"/>
+    </geometry>
+  </collision>
+</link>
+<link name="shoulder_v2_1">
+  <inertial>
+    <origin xyz="-0.05003301392386567 0.00744711420020433 0.06537453945113983" rpy="0 0 0"/>
+    <mass value="0.7582173734794716"/>
+    <inertia ixx="0.001635" iyy="0.002653" izz="0.001251" ixy="0.0" iyz="0.000136" ixz="-1e-06"/>
+  </inertial>
+  <visual>
+    <origin xyz="-0.05 0.095 -0.1504" rpy="0 0 0"/>
+    <geometry>
+      <mesh filename="file://$(find arm_description)/meshes/shoulder_v2_1.stl" scale="0.001 0.001 0.001"/>
+    </geometry>
+    <material name="blue"/>
+  </visual>
+  <collision>
+    <origin xyz="-0.05 0.095 -0.1504" rpy="0 0 0"/>
+    <geometry>
+      <mesh filename="file://$(find arm_description)/meshes/shoulder_v2_1.stl" scale="0.001 0.001 0.001"/>
+    </geometry>
+  </collision>
+</link>
+<link name="plangearbox1_v2_1">
+  <inertial>
+    <origin xyz="-2.198402479996289e-05 0.04289853923367516 7.979625855469852e-06" rpy="0 0 0"/>
+    <mass value="2.0006291062763104"/>
+    <inertia ixx="0.001765" iyy="0.000982" izz="0.001764" ixy="0.0" iyz="1e-06" ixz="-0.0"/>
+  </inertial>
+  <visual>
+    <origin xyz="2.4e-05 0.097184 -0.1954" rpy="0 0 0"/>
+    <geometry>
+      <mesh filename="file://$(find arm_description)/meshes/plangearbox1_v2_1.stl" scale="0.001 0.001 0.001"/>
+    </geometry>
+    <material name="black"/>
+  </visual>
+  <collision>
+    <origin xyz="2.4e-05 0.097184 -0.1954" rpy="0 0 0"/>
+    <geometry>
+      <mesh filename="file://$(find arm_description)/meshes/plangearbox1_v2_1.stl" scale="0.001 0.001 0.001"/>
+    </geometry>
+  </collision>
+</link>
+<link name="stepper1_v2_1">
+  <inertial>
+    <origin xyz="-2.2452245726494987e-05 0.04805206213786515 3.443202523836786e-05" rpy="0 0 0"/>
+    <mass value="0.47672097000804026"/>
+    <inertia ixx="0.000488" iyy="0.000235" izz="0.000488" ixy="0.0" iyz="-1e-06" ixz="-0.0"/>
+  </inertial>
+  <visual>
+    <origin xyz="6.7e-05 0.013684 -0.1954" rpy="0 0 0"/>
+    <geometry>
+      <mesh filename="file://$(find arm_description)/meshes/stepper1_v2_1.stl" scale="0.001 0.001 0.001"/>
+    </geometry>
+    <material name="black"/>
+  </visual>
+  <collision>
+    <origin xyz="6.7e-05 0.013684 -0.1954" rpy="0 0 0"/>
+    <geometry>
+      <mesh filename="file://$(find arm_description)/meshes/stepper1_v2_1.stl" scale="0.001 0.001 0.001"/>
+    </geometry>
+  </collision>
+</link>
+<link name="shoulder_bearling_house2_prt3_v3_1">
+  <inertial>
+    <origin xyz="-4.0536114861531317e-07 -0.0059858275962992105 -9.453793303748625e-11" rpy="0 0 0"/>
+    <mass value="0.05938208856291783"/>
+    <inertia ixx="3.7e-05" iyy="7.3e-05" izz="3.7e-05" ixy="-0.0" iyz="0.0" ixz="0.0"/>
+  </inertial>
+  <visual>
+    <origin xyz="4.5e-05 0.055884 -0.2754" rpy="0 0 0"/>
+    <geometry>
+      <mesh filename="file://$(find arm_description)/meshes/shoulder_bearling_house2_prt3_v3_1.stl" scale="0.001 0.001 0.001"/>
+    </geometry>
+    <material name="blue"/>
+  </visual>
+  <collision>
+    <origin xyz="4.5e-05 0.055884 -0.2754" rpy="0 0 0"/>
+    <geometry>
+      <mesh filename="file://$(find arm_description)/meshes/shoulder_bearling_house2_prt3_v3_1.stl" scale="0.001 0.001 0.001"/>
+    </geometry>
+  </collision>
+</link>
+<link name="new_pipe_b_v8_1">
+  <inertial>
+    <origin xyz="-3.1295264940206456e-05 0.05999962743199911 0.002489679948011303" rpy="0 0 0"/>
+    <mass value="0.08655426473406591"/>
+    <inertia ixx="0.000229" iyy="3.8e-05" izz="0.000226" ixy="0.0" iyz="-0.0" ixz="-0.0"/>
+  </inertial>
+  <visual>
+    <origin xyz="2.1e-05 0.102029 -0.2754" rpy="0 0 0"/>
+    <geometry>
+      <mesh filename="file://$(find arm_description)/meshes/new_pipe_b_v8_1.stl" scale="0.001 0.001 0.001"/>
+    </geometry>
+    <material name="black"/>
+  </visual>
+  <collision>
+    <origin xyz="2.1e-05 0.102029 -0.2754" rpy="0 0 0"/>
+    <geometry>
+      <mesh filename="file://$(find arm_description)/meshes/new_pipe_b_v8_1.stl" scale="0.001 0.001 0.001"/>
+    </geometry>
+  </collision>
+</link>
+<link name="shoulder_bearling_house_2prt1_v5_1">
+  <inertial>
+    <origin xyz="4.24595728622469e-06 -0.004300516777600696 -4.207479079365584e-06" rpy="0 0 0"/>
+    <mass value="0.05778324976734234"/>
+    <inertia ixx="3.6e-05" iyy="7.1e-05" izz="3.6e-05" ixy="-0.0" iyz="-0.0" ixz="0.0"/>
+  </inertial>
+  <visual>
+    <origin xyz="2.1e-05 0.102029 -0.2754" rpy="0 0 0"/>
+    <geometry>
+      <mesh filename="file://$(find arm_description)/meshes/shoulder_bearling_house_2prt1_v5_1.stl" scale="0.001 0.001 0.001"/>
+    </geometry>
+    <material name="blue"/>
+  </visual>
+  <collision>
+    <origin xyz="2.1e-05 0.102029 -0.2754" rpy="0 0 0"/>
+    <geometry>
+      <mesh filename="file://$(find arm_description)/meshes/shoulder_bearling_house_2prt1_v5_1.stl" scale="0.001 0.001 0.001"/>
+    </geometry>
+  </collision>
+</link>
+<link name="shoulder_bearling_house2_prt2_v10_1">
+  <inertial>
+    <origin xyz="-7.534969931434021e-06 0.00999965589472103 7.596384632435615e-11" rpy="0 0 0"/>
+    <mass value="0.17595730314710867"/>
+    <inertia ixx="0.000105" iyy="0.000198" izz="0.000105" ixy="-0.0" iyz="0.0" ixz="-0.0"/>
+  </inertial>
+  <visual>
+    <origin xyz="3e-05 0.085884 -0.2754" rpy="0 0 0"/>
+    <geometry>
+      <mesh filename="file://$(find arm_description)/meshes/shoulder_bearling_house2_prt2_v10_1.stl" scale="0.001 0.001 0.001"/>
+    </geometry>
+    <material name="blue"/>
+  </visual>
+  <collision>
+    <origin xyz="3e-05 0.085884 -0.2754" rpy="0 0 0"/>
+    <geometry>
+      <mesh filename="file://$(find arm_description)/meshes/shoulder_bearling_house2_prt2_v10_1.stl" scale="0.001 0.001 0.001"/>
+    </geometry>
+  </collision>
+</link>
+<link name="tbone_v1_1">
+  <inertial>
+    <origin xyz="-0.0001179461306405897 -0.040037043730441445 0.011561726312559306" rpy="0 0 0"/>
+    <mass value="0.7230946223073603"/>
+    <inertia ixx="0.000893" iyy="0.000815" izz="0.000779" ixy="0.0" iyz="-0.0" ixz="-1e-06"/>
+  </inertial>
+  <visual>
+    <origin xyz="9.6e-05 -0.042971 -0.2754" rpy="0 0 0"/>
+    <geometry>
+      <mesh filename="file://$(find arm_description)/meshes/tbone_v1_1.stl" scale="0.001 0.001 0.001"/>
+    </geometry>
+    <material name="blue"/>
+  </visual>
+  <collision>
+    <origin xyz="9.6e-05 -0.042971 -0.2754" rpy="0 0 0"/>
+    <geometry>
+      <mesh filename="file://$(find arm_description)/meshes/tbone_v1_1.stl" scale="0.001 0.001 0.001"/>
+    </geometry>
+  </collision>
+</link>
+<link name="pipe_c_v1_1">
+  <inertial>
+    <origin xyz="-0.00013201873724399225 0.004305319532101214 0.029999580087758992" rpy="0 0 0"/>
+    <mass value="0.03153060769791503"/>
+    <inertia ixx="1.6e-05" iyy="1.5e-05" izz="1.2e-05" ixy="0.0" iyz="0.0" ixz="0.0"/>
+  </inertial>
+  <visual>
+    <origin xyz="0.0002 -0.002971 -0.308202" rpy="0 0 0"/>
+    <geometry>
+      <mesh filename="file://$(find arm_description)/meshes/pipe_c_v1_1.stl" scale="0.001 0.001 0.001"/>
+    </geometry>
+    <material name="black"/>
+  </visual>
+  <collision>
+    <origin xyz="0.0002 -0.002971 -0.308202" rpy="0 0 0"/>
+    <geometry>
+      <mesh filename="file://$(find arm_description)/meshes/pipe_c_v1_1.stl" scale="0.001 0.001 0.001"/>
+    </geometry>
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