Commit message: updated link names and added colors in gazebo

File: robot_base_description/urdf/robot_base.xacro (robot description, xacro)
@@ -24,5 +24,5 @@
   </collision>
 </link>
-<link name="left_front_wheel_1">
+<link name="left_front_wheel">
   <inertial>
     <origin xyz="-9.543055706773274e-09 0.03137916494591725 1.4559213505627167e-07" rpy="0 0 0"/>
@@ -33,5 +33,5 @@
     <origin xyz="-0.19 -0.1805 -0.08" rpy="0 0 0"/>
     <geometry>
-      <mesh filename="file://$(find robot_base_description)/meshes/left_front_wheel_1.stl" scale="0.001 0.001 0.001"/>
+      <mesh filename="file://$(find robot_base_description)/meshes/left_front_wheel.stl" scale="0.001 0.001 0.001"/>
     </geometry>
     <material name="silver"/>
@@ -40,9 +40,9 @@
     <origin xyz="-0.19 -0.1805 -0.08" rpy="0 0 0"/>
     <geometry>
-      <mesh filename="file://$(find robot_base_description)/meshes/left_front_wheel_1.stl" scale="0.001 0.001 0.001"/>
-    </geometry>
-  </collision>
-</link>
-<link name="left_back_wheel_1">
+      <mesh filename="file://$(find robot_base_description)/meshes/left_front_wheel.stl" scale="0.001 0.001 0.001"/>
+    </geometry>
+  </collision>
+</link>
+<link name="left_back_wheel">
   <inertial>
     <origin xyz="-9.543055595750971e-09 0.03137916494591733 1.4559213526443848e-07" rpy="0 0 0"/>
@@ -53,5 +53,5 @@
     <origin xyz="0.19 -0.1805 -0.08" rpy="0 0 0"/>
     <geometry>
-      <mesh filename="file://$(find robot_base_description)/meshes/left_back_wheel_1.stl" scale="0.001 0.001 0.001"/>
+      <mesh filename="file://$(find robot_base_description)/meshes/left_back_wheel.stl" scale="0.001 0.001 0.001"/>
     </geometry>
     <material name="silver"/>
@@ -60,9 +60,9 @@
     <origin xyz="0.19 -0.1805 -0.08" rpy="0 0 0"/>
     <geometry>
-      <mesh filename="file://$(find robot_base_description)/meshes/left_back_wheel_1.stl" scale="0.001 0.001 0.001"/>
-    </geometry>
-  </collision>
-</link>
-<link name="right_back_wheel_1">
+      <mesh filename="file://$(find robot_base_description)/meshes/left_back_wheel.stl" scale="0.001 0.001 0.001"/>
+    </geometry>
+  </collision>
+</link>
+<link name="right_back_wheel">
   <inertial>
     <origin xyz="2.3498597973015123e-07 -0.03137920521938581 -2.0518912122180488e-07" rpy="0 0 0"/>
@@ -73,5 +73,5 @@
     <origin xyz="0.19 0.1805 -0.08" rpy="0 0 0"/>
     <geometry>
-      <mesh filename="file://$(find robot_base_description)/meshes/right_back_wheel_1.stl" scale="0.001 0.001 0.001"/>
+      <mesh filename="file://$(find robot_base_description)/meshes/right_back_wheel.stl" scale="0.001 0.001 0.001"/>
     </geometry>
     <material name="silver"/>
@@ -80,9 +80,9 @@
     <origin xyz="0.19 0.1805 -0.08" rpy="0 0 0"/>
     <geometry>
-      <mesh filename="file://$(find robot_base_description)/meshes/right_back_wheel_1.stl" scale="0.001 0.001 0.001"/>
-    </geometry>
-  </collision>
-</link>
-<link name="right_front_wheel_1">
+      <mesh filename="file://$(find robot_base_description)/meshes/right_back_wheel.stl" scale="0.001 0.001 0.001"/>
+    </geometry>
+  </collision>
+</link>
+<link name="right_front_wheel">
   <inertial>
     <origin xyz="2.3498597989668468e-07 -0.03137920521938581 -2.0518912093037134e-07" rpy="0 0 0"/>
@@ -93,5 +93,5 @@
     <origin xyz="-0.19 0.1805 -0.08" rpy="0 0 0"/>
     <geometry>
-      <mesh filename="file://$(find robot_base_description)/meshes/right_front_wheel_1.stl" scale="0.001 0.001 0.001"/>
+      <mesh filename="file://$(find robot_base_description)/meshes/right_front_wheel.stl" scale="0.001 0.001 0.001"/>
     </geometry>
     <material name="silver"/>
@@ -100,9 +100,9 @@
     <origin xyz="-0.19 0.1805 -0.08" rpy="0 0 0"/>
     <geometry>
-      <mesh filename="file://$(find robot_base_description)/meshes/right_front_wheel_1.stl" scale="0.001 0.001 0.001"/>
-    </geometry>
-  </collision>
-</link>
-<link name="zed_mini_1">
+      <mesh filename="file://$(find robot_base_description)/meshes/right_front_wheel.stl" scale="0.001 0.001 0.001"/>
+    </geometry>
+  </collision>
+</link>
+<link name="zed_mini">
   <inertial>
     <origin xyz="0.006890809169695311 -0.0011814639225888749 0.013252607692305629" rpy="0 0 0"/>
@@ -113,5 +113,5 @@
     <origin xyz="-0.2525 -0.0 -0.1085" rpy="0 0 0"/>
     <geometry>
-      <mesh filename="file://$(find robot_base_description)/meshes/zed_mini_1.stl" scale="0.001 0.001 0.001"/>
+      <mesh filename="file://$(find robot_base_description)/meshes/zed_mini.stl" scale="0.001 0.001 0.001"/>
     </geometry>
     <material name="silver"/>
@@ -120,9 +120,9 @@
     <origin xyz="-0.2525 -0.0 -0.1085" rpy="0 0 0"/>
     <geometry>
-      <mesh filename="file://$(find robot_base_description)/meshes/zed_mini_1.stl" scale="0.001 0.001 0.001"/>
-    </geometry>
-  </collision>
-</link>
-<link name="logo_1">
+      <mesh filename="file://$(find robot_base_description)/meshes/zed_mini.stl" scale="0.001 0.001 0.001"/>
+    </geometry>
+  </collision>
+</link>
+<link name="logo">
   <inertial>
     <origin xyz="-0.0030148374702534397 -0.0009578344360897588 -0.0011300936134206602" rpy="0 0 0"/>
@@ -133,5 +133,5 @@
     <origin xyz="-0.26 -0.0 -0.08975" rpy="0 0 0"/>
     <geometry>
-      <mesh filename="file://$(find robot_base_description)/meshes/logo_1.stl" scale="0.001 0.001 0.001"/>
+      <mesh filename="file://$(find robot_base_description)/meshes/logo.stl" scale="0.001 0.001 0.001"/>
     </geometry>
     <material name="silver"/>
@@ -140,9 +140,9 @@
     <origin xyz="-0.26 -0.0 -0.08975" rpy="0 0 0"/>
     <geometry>
-      <mesh filename="file://$(find robot_base_description)/meshes/logo_1.stl" scale="0.001 0.001 0.001"/>
-    </geometry>
-  </collision>
-</link>
-<link name="jetson_1">
+      <mesh filename="file://$(find robot_base_description)/meshes/logo.stl" scale="0.001 0.001 0.001"/>
+    </geometry>
+  </collision>
+</link>
+<link name="jetson">
   <inertial>
     <origin xyz="-0.001882812378843579 -0.0012117915536683699 0.009224709951320367" rpy="0 0 0"/>
@@ -153,5 +153,5 @@
     <origin xyz="0.230479 -0.0 -0.108" rpy="0 0 0"/>
     <geometry>
-      <mesh filename="file://$(find robot_base_description)/meshes/jetson_1.stl" scale="0.001 0.001 0.001"/>
+      <mesh filename="file://$(find robot_base_description)/meshes/jetson.stl" scale="0.001 0.001 0.001"/>
     </geometry>
     <material name="silver"/>
@@ -160,9 +160,9 @@
     <origin xyz="0.230479 -0.0 -0.108" rpy="0 0 0"/>
     <geometry>
-      <mesh filename="file://$(find robot_base_description)/meshes/jetson_1.stl" scale="0.001 0.001 0.001"/>
-    </geometry>
-  </collision>
-</link>
-<link name="lidar_1">
+      <mesh filename="file://$(find robot_base_description)/meshes/jetson.stl" scale="0.001 0.001 0.001"/>
+    </geometry>
+  </collision>
+</link>
+<link name="lidar">
   <inertial>
     <origin xyz="0.041705900429680434 -3.652874609497409e-17 0.03970114222279103" rpy="0 0 0"/>
@@ -173,5 +173,5 @@
     <origin xyz="-0.0 -0.0 -0.141" rpy="0 0 0"/>
     <geometry>
-      <mesh filename="file://$(find robot_base_description)/meshes/lidar_1.stl" scale="0.001 0.001 0.001"/>
+      <mesh filename="file://$(find robot_base_description)/meshes/lidar.stl" scale="0.001 0.001 0.001"/>
     </geometry>
     <material name="silver"/>
@@ -180,9 +180,9 @@
     <origin xyz="-0.0 -0.0 -0.141" rpy="0 0 0"/>
     <geometry>
-      <mesh filename="file://$(find robot_base_description)/meshes/lidar_1.stl" scale="0.001 0.001 0.001"/>
-    </geometry>
-  </collision>
-</link>
-<link name="imu_1">
+      <mesh filename="file://$(find robot_base_description)/meshes/lidar.stl" scale="0.001 0.001 0.001"/>
+    </geometry>
+  </collision>
+</link>
+<link name="imu">
   <inertial>
     <origin xyz="-0.00998812297806373 9.133494040341156e-05 0.000862164665477741" rpy="0 0 0"/>
@@ -193,5 +193,5 @@
     <origin xyz="0.164479 -0.0 -0.108" rpy="0 0 0"/>
     <geometry>
-      <mesh filename="file://$(find robot_base_description)/meshes/imu_1.stl" scale="0.001 0.001 0.001"/>
+      <mesh filename="file://$(find robot_base_description)/meshes/imu.stl" scale="0.001 0.001 0.001"/>
     </geometry>
     <material name="silver"/>
@@ -200,5 +200,5 @@
     <origin xyz="0.164479 -0.0 -0.108" rpy="0 0 0"/>
     <geometry>
-      <mesh filename="file://$(find robot_base_description)/meshes/imu_1.stl" scale="0.001 0.001 0.001"/>
+      <mesh filename="file://$(find robot_base_description)/meshes/imu.stl" scale="0.001 0.001 0.001"/>
     </geometry>
   </collision>
@@ -207,5 +207,5 @@
   <origin xyz="0.19 0.1805 0.08" rpy="0 0 0"/>
   <parent link="base_link"/>
-  <child link="left_front_wheel_1"/>
+  <child link="left_front_wheel"/>
   <axis xyz="0.0 1.0 0.0"/>
 </joint>
@@ -213,5 +213,5 @@
   <origin xyz="-0.19 0.1805 0.08" rpy="0 0 0"/>
   <parent link="base_link"/>
-  <child link="left_back_wheel_1"/>
+  <child link="left_back_wheel"/>
   <axis xyz="0.0 1.0 0.0"/>
 </joint>
@@ -219,5 +219,5 @@
   <origin xyz="-0.19 -0.1805 0.08" rpy="0 0 0"/>
   <parent link="base_link"/>
-  <child link="right_back_wheel_1"/>
+  <child link="right_back_wheel"/>
   <axis xyz="0.0 -1.0 0.0"/>
 </joint>
@@ -225,5 +225,5 @@
   <origin xyz="0.19 -0.1805 0.08" rpy="0 0 0"/>
   <parent link="base_link"/>
-  <child link="right_front_wheel_1"/>
+  <child link="right_front_wheel"/>
   <axis xyz="0.0 -1.0 0.0"/>
 </joint>
@@ -231,25 +231,115 @@
   <origin xyz="0.2525 0.0 0.1085" rpy="0 0 0"/>
   <parent link="base_link"/>
-  <child link="zed_mini_1"/>
+  <child link="zed_mini"/>
 </joint>
 <joint name="logo_joint" type="fixed">
   <origin xyz="0.26 0.0 0.08975" rpy="0 0 0"/>
   <parent link="base_link"/>
-  <child link="logo_1"/>
+  <child link="logo"/>
 </joint>
 <joint name="jetson_joint" type="fixed">
   <origin xyz="-0.230479 0.0 0.108" rpy="0 0 0"/>
   <parent link="base_link"/>
-  <child link="jetson_1"/>
+  <child link="jetson"/>
 </joint>
 <joint name="lidar_joint" type="fixed">
   <origin xyz="0.0 0.0 0.141" rpy="0 0 0"/>
   <parent link="base_link"/>
-  <child link="lidar_1"/>
+  <child link="lidar"/>
 </joint>
 <joint name="imu_joint" type="fixed">
   <origin xyz="-0.164479 0.0 0.108" rpy="0 0 0"/>
   <parent link="base_link"/>
-  <child link="imu_1"/>
-</joint>
+  <child link="imu"/>
+</joint>
+<gazebo reference="base_link">
+    <visual>
+    <material>
+        <ambient>1.0 0.0 0.0 1.0</ambient>
+        <diffuse>1.0 0.0 0.0 1.0</diffuse>
+        <specular>1.0 0.0 0.0 1.0</specular>
+    </material>
+    </visual>
+</gazebo>
+<gazebo reference="left_front_wheel">
+    <visual>
+    <material>
+        <ambient>0.0 0.0 0.0 1.0</ambient>
+        <diffuse>0.0 0.0 0.0 1.0</diffuse>
+        <specular>0.0 0.0 0.0 1.0</specular>
+    </material>
+    </visual>
+</gazebo>
+<gazebo reference="left_back_wheel">
+    <visual>
+    <material>
+        <ambient>0.0 0.0 0.0 1.0</ambient>
+        <diffuse>0.0 0.0 0.0 1.0</diffuse>
+        <specular>0.0 0.0 0.0 1.0</specular>
+    </material>
+    </visual>
+</gazebo>
+<gazebo reference="right_front_wheel">
+    <visual>
+    <material>
+        <ambient>0.0 0.0 0.0 1.0</ambient>
+        <diffuse>0.0 0.0 0.0 1.0</diffuse>
+        <specular>0.0 0.0 0.0 1.0</specular>
+    </material>
+    </visual>
+</gazebo>
+<gazebo reference="right_back_wheel">
+    <visual>
+    <material>
+        <ambient>0.0 0.0 0.0 1.0</ambient>
+        <diffuse>0.0 0.0 0.0 1.0</diffuse>
+        <specular>0.0 0.0 0.0 1.0</specular>
+    </material>
+    </visual>
+</gazebo>
+<gazebo reference="logo">
+    <visual>
+    <material>
+        <ambient>0.0 0.0 0.0 1.0</ambient>
+        <diffuse>0.0 0.0 0.0 1.0</diffuse>
+        <specular>0.0 0.0 0.0 1.0</specular>
+    </material>
+    </visual>
+</gazebo>
+<gazebo reference="lidar">
+    <visual>
+    <material>
+        <ambient>0.0 0.0 1.0 1.0</ambient>
+        <diffuse>0.0 0.0 1.0 1.0</diffuse>
+        <specular>0.0 0.0 1.0 1.0</specular>
+    </material>
+    </visual>
+</gazebo>
+<gazebo reference="imu">
+    <visual>
+    <material>
+        <ambient>0.0 1.0 0.0 1.0</ambient>
+        <diffuse>0.0 1.0 0.0 1.0</diffuse>
+        <specular>0.0 1.0 0.0 1.0</specular>
+    </material>
+    </visual>
+</gazebo>
+<gazebo reference="jetson">
+    <visual>
+    <material>
+        <ambient>0.0 1.0 0.0 1.0</ambient>
+        <diffuse>0.0 1.0 0.0 1.0</diffuse>
+        <specular>0.0 1.0 0.0 1.0</specular>
+    </material>
+    </visual>
+</gazebo>
+<gazebo reference="zed_mini">
+    <visual>
+    <material>
+        <ambient>0.752 0.752 0.752 1.0</ambient>
+        <diffuse>0.752 0.752 0.752 1.0</diffuse>
+        <specular>0.752 0.752 0.752 1.0</specular>
+    </material>
+    </visual>
+</gazebo>
 </robot>

Commit message: Add files via upload

File: robot_base_description/urdf/robot_base.xacro (robot description, xacro)
@@ -1220,5 +1220,5 @@
   </collision>
 </link>
-<joint name="left_front_joint" type="continuous">
+<joint name="left_front_wheel_joint" type="continuous">
   <origin xyz="0.19 0.1805 0.08" rpy="0 0 0"/>
   <parent link="base_link"/>
@@ -1226,5 +1226,5 @@
   <axis xyz="0.0 1.0 0.0"/>
 </joint>
-<joint name="left_back_joint" type="continuous">
+<joint name="left_back_wheel_joint" type="continuous">
   <origin xyz="-0.19 0.1805 0.08" rpy="0 0 0"/>
   <parent link="base_link"/>
@@ -1232,5 +1232,5 @@
   <axis xyz="0.0 1.0 0.0"/>
 </joint>
-<joint name="right_front_joint" type="continuous">
+<joint name="right_front_wheel_joint" type="continuous">
   <origin xyz="0.19 -0.1805 0.08" rpy="0 0 0"/>
   <parent link="base_link"/>
@@ -1238,5 +1238,5 @@
   <axis xyz="0.0 1.0 0.0"/>
 </joint>
-<joint name="right_back_joint" type="continuous">
+<joint name="right_back_wheel_joint" type="continuous">
   <origin xyz="-0.19 -0.1805 0.08" rpy="0 0 0"/>
   <parent link="base_link"/>

File: robot_base_description/urdf/ros2_control.xacro (robot description, xacro)
@@ -5,6 +5,6 @@
       <hardware>
         <plugin>hoverboard_hardware_interface/HoverboardHardwareInterface</plugin>
-        <param name="left_wheel_joint_name">left_front_wheel_joint</param>
-        <param name="right_wheel_joint_name">right_front_wheel_joint</param>
+        <param name="left_front_wheel_joint_name">left_front_wheel_joint</param>
+        <param name="right_front_wheel_joint_name">right_front_wheel_joint</param>
         <param name="loop_rate">50</param>
         <param name="device">/dev/ttyUSB0</param>

Commit message: Add files via upload

File: robot_base_description/urdf/robot_base.xacro (robot description, xacro)
@@ -5,4 +5,12 @@
 <xacro:include filename="$(find robot_base_description)/urdf/ros2_control.xacro" />
 <xacro:include filename="$(find robot_base_description)/urdf/robot_base.gazebo" />
+<!-- Define the front and back serial devices -->
+  <xacro:property name="front_device" value="/dev/ttyUSB0"/>
+  <xacro:property name="back_device" value="/dev/ttyUSB1"/>
+<!-- Include the hoverboard_ros2_control macro with front and back devices -->
+  <xacro:macro name="include_hoverboard_ros2_control" params="front_device back_device">
+  <xacro:hoverboard_ros2_control name="Hoverboard_robot" front_device="${front_device}" back_device="${back_device}"/>
+  </xacro:macro>
+<xacro:include_hoverboard_ros2_control front_device="${front_device}" back_device="${back_device}"/>
 <link name="base_link">
   <visual>
@@ -1530,4 +1538,4 @@
   <child link="shoulder_bearling_house_prt2_v1_1"/>
 </joint>
-<xacro:hoverboard_ros2_control name="Hoverboard" />
+<xacro:hoverboard_ros2_control name="Hoverboard" front_device="$(front_device)" back_device="$(back_device)"/>
 </robot>

File: robot_base_description/urdf/ros2_control.xacro (robot description, xacro)
@@ -5,18 +5,31 @@
       <hardware>
         <plugin>hoverboard_hardware_interface/HoverboardHardwareInterface</plugin>
-        <param name="left_front_wheel_joint_name">left_front_wheel_joint</param>
-        <param name="right_front_wheel_joint_name">right_front_wheel_joint</param>
+        <param name="front_left_wheel_joint_name">front_left_wheel_joint</param>
+        <param name="front_right_wheel_joint_name">front_right_wheel_joint</param>
+        <param name="back_left_wheel_joint_name">back_left_wheel_joint</param>
+        <param name="back_right_wheel_joint_name">back_right_wheel_joint</param>
         <param name="loop_rate">50</param>
-        <param name="device">/dev/ttyUSB0</param>
+        <param name="front_device">${front_device}</param>
+        <param name="back_device">${back_device}</param>
         <param name="baud_rate">115200</param>
         <param name="timeout">1000</param>
         <param name="encoder_ticks_per_revolution">90</param>
       </hardware>
-      <joint name="left_front_wheel_joint">
+      <joint name="front_left_wheel_joint">
         <command_interface name="velocity"/>
         <state_interface name="position"/>
         <state_interface name="velocity"/>
       </joint>
-      <joint name="right_front_wheel_joint">
+      <joint name="front_right_wheel_joint">
+        <command_interface name="velocity"/>
+        <state_interface name="position"/>
+        <state_interface name="velocity"/>
+      </joint>
+      <joint name="back_left_wheel_joint">
+        <command_interface name="velocity"/>
+        <state_interface name="position"/>
+        <state_interface name="velocity"/>
+      </joint>
+      <joint name="back_right_wheel_joint">
         <command_interface name="velocity"/>
         <state_interface name="position"/>

Commit message: Add files via upload

File: robot_base_description/urdf/robot_base.xacro (robot description, xacro)
@@ -5,12 +5,13 @@
 <xacro:include filename="$(find robot_base_description)/urdf/ros2_control.xacro" />
 <xacro:include filename="$(find robot_base_description)/urdf/robot_base.gazebo" />
-<!-- Define the front and back serial devices -->
+<!-- Define the front and back serial devices
   <xacro:property name="front_device" value="/dev/ttyUSB0"/>
-  <xacro:property name="back_device" value="/dev/ttyUSB1"/>
-<!-- Include the hoverboard_ros2_control macro with front and back devices -->
+  <xacro:property name="back_device" value="/dev/ttyUSB1"/>  -->
+<!-- Include the hoverboard_ros2_control macro with front and back devices
   <xacro:macro name="include_hoverboard_ros2_control" params="front_device back_device">
-  <xacro:hoverboard_ros2_control name="Hoverboard_robot" front_device="${front_device}" back_device="${back_device}"/>
+  <xacro:hoverboard_ros2_control name="hoverboard_ros2_control" front_device="${front_device}" back_device="${back_device}"/>
   </xacro:macro>
-<xacro:include_hoverboard_ros2_control front_device="${front_device}" back_device="${back_device}"/>
+ <xacro:include_hoverboard_ros2_control front_device="${front_device}" back_device="${back_device}"/>
+  -->
 <link name="base_link">
   <visual>
@@ -1538,4 +1539,5 @@
   <child link="shoulder_bearling_house_prt2_v1_1"/>
 </joint>
-<xacro:hoverboard_ros2_control name="Hoverboard" front_device="$(front_device)" back_device="$(back_device)"/>
+<xacro:hoverboard_ros2_control name="Hoverboard" />
+<!-- <xacro:include_hoverboard_ros2_control front_device="${front_device}" back_device="${back_device}"/> -->
 </robot>

File: robot_base_description/urdf/ros2_control.xacro (robot description, xacro)
@@ -5,31 +5,31 @@
       <hardware>
         <plugin>hoverboard_hardware_interface/HoverboardHardwareInterface</plugin>
-        <param name="front_left_wheel_joint_name">front_left_wheel_joint</param>
-        <param name="front_right_wheel_joint_name">front_right_wheel_joint</param>
-        <param name="back_left_wheel_joint_name">back_left_wheel_joint</param>
-        <param name="back_right_wheel_joint_name">back_right_wheel_joint</param>
-        <param name="loop_rate">50</param>
-        <param name="front_device">${front_device}</param>
-        <param name="back_device">${back_device}</param>
+        <param name="left_front_wheel_joint_name">left_front_wheel_joint</param>
+        <param name="right_front_wheel_joint_name">right_front_wheel_joint</param>
+        <param name="left_back_wheel_joint_name">left_back_wheel_joint</param>
+        <param name="right_back_wheel_joint_name">right_back_wheel_joint</param>
+        <param name="loop_rate">100</param>
+        <param name="front_device">/dev/ttyUSB0</param>
+        <param name="back_device">/dev/ttyUSB1</param>
         <param name="baud_rate">115200</param>
         <param name="timeout">1000</param>
         <param name="encoder_ticks_per_revolution">90</param>
       </hardware>
-      <joint name="front_left_wheel_joint">
+      <joint name="left_front_wheel_joint">
         <command_interface name="velocity"/>
         <state_interface name="position"/>
         <state_interface name="velocity"/>
       </joint>
-      <joint name="front_right_wheel_joint">
+      <joint name="right_front_wheel_joint">
         <command_interface name="velocity"/>
         <state_interface name="position"/>
         <state_interface name="velocity"/>
       </joint>
-      <joint name="back_left_wheel_joint">
+      <joint name="left_back_wheel_joint">
         <command_interface name="velocity"/>
         <state_interface name="position"/>
         <state_interface name="velocity"/>
       </joint>
-      <joint name="back_right_wheel_joint">
+      <joint name="right_back_wheel_joint">
         <command_interface name="velocity"/>
         <state_interface name="position"/>
