Commit message: Add files via upload

File: robot_base_description/urdf/ros2_control.xacro (robot description, xacro)
@@ -2,11 +2,11 @@
 <robot xmlns:xacro="http://www.ros.org/wiki/xacro">
   <xacro:macro name="hoverboard_ros2_control" params="name">
-    <ros2_control name="${name}" type="system">
+      <ros2_control name="${name}_front" type="system">
       <hardware>
         <plugin>hoverboard_hardware_interface/HoverboardHardwareInterface</plugin>
-        <param name="left_wheel_joint_name">left_front_wheel_joint</param>
-        <param name="right_wheel_joint_name">right_front_wheel_joint</param>
-        <param name="loop_rate">50</param>
-        <param name="device">/dev/ttyUSB0</param>
+        <param name="left_front_wheel_joint_name">left_front_wheel_joint</param>
+        <param name="right_front_wheel_joint_name">right_front_wheel_joint</param>
+        <param name="loop_rate">100</param>
+        <param name="front_device">/dev/ttyUSB0</param>
         <param name="baud_rate">115200</param>
         <param name="timeout">1000</param>
@@ -23,5 +23,27 @@
         <state_interface name="velocity"/>
       </joint>
-    </ros2_control>
+      </ros2_control>
+      <ros2_control name="${name}_back" type="system">
+      <hardware>
+        <plugin>hoverboard_hardware_interface/HoverboardHardwareInterface</plugin>
+        <param name="left_back_wheel_joint_name">left_back_wheel_joint</param>
+        <param name="right_back_wheel_joint_name">right_back_wheel_joint</param>
+        <param name="loop_rate">100</param>
+        <param name="back_device">/dev/ttyUSB1</param>
+        <param name="baud_rate">115200</param>
+        <param name="timeout">1000</param>
+        <param name="encoder_ticks_per_revolution">90</param>
+      </hardware>
+      <joint name="left_back_wheel_joint">
+        <command_interface name="velocity"/>
+        <state_interface name="position"/>
+        <state_interface name="velocity"/>
+      </joint>
+      <joint name="right_back_wheel_joint">
+        <command_interface name="velocity"/>
+        <state_interface name="position"/>
+        <state_interface name="velocity"/>
+      </joint>
+      </ros2_control>
   </xacro:macro>
 </robot>
