Commit message: Add files via upload

File: hoverboard_ros2_control/hoverboard_demo_description/urdf/hoverboard_description.xacro (robot description, xacro)
@@ -15,4 +15,6 @@
     <xacro:property name="caster_wheel_weight" value="0.1" />
     <link name="base_link">
+    </link>
+    <link name="base_footprint">
     </link>
     <link name="plate">
@@ -177,4 +179,9 @@
         <child link="plate" />
     </joint>
+    <joint name="base_link_print_joint" type="fixed">
+        <origin rpy="0 0 0" xyz="0 0 0" />
+        <parent link="base_link" />
+        <child link="base_footprint" />
+    </joint>
     <joint name="lidar_joint" type="fixed">
   <origin xyz="0.0 0.0 0.141" rpy="0 0 0"/>

File: hoverboard_ros2_control/hoverboard_demo_description/urdf/ros2_control.xacro (robot description, xacro)
@@ -7,5 +7,5 @@
         <param name="left_wheel_joint_name">driving_wheel_front_left_joint</param>
         <param name="right_wheel_joint_name">driving_wheel_front_right_joint</param>
-        <param name="loop_rate">50</param>
+        <param name="loop_rate">40</param>
         <param name="device">/dev/ttyUSB0</param>
         <param name="baud_rate">115200</param>
@@ -29,5 +29,5 @@
         <param name="left_wheel_joint_name">driving_wheel_back_left_joint</param>
         <param name="right_wheel_joint_name">driving_wheel_back_right_joint</param>
-        <param name="loop_rate">50</param>
+        <param name="loop_rate">40</param>
         <param name="device">/dev/ttyUSB1</param>
         <param name="baud_rate">115200</param>
